File: PCB/_autosave-hackpad.kicad_pcb (KiCad board)
At the start: 2 copper layers, 61.9 x 40.5 mm, 8 parts, among them SW1 SW_Push, SW2 SW_Push, SW3 SW_Push, SW4 SW_Push, U1 XIAO-RP2040-DIP

Commit message: updated
Other:
- board size 61.9 x 40.5 mm -> 61.9 x 38.1 mm
Changed lines of the file:
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@@
 			(outputformat 1)
 			(mirror no)
-			(drillshape 0)
+			(drillshape 1)
 			(scaleselection 1)
-			(outputdirectory "../Production/")
+			(outputdirectory "")
 		)
 	)
@@
 	)
 	(gr_rect
-		(start 109.5375 23.8125)
+		(start 109.5375 26.19375)
 		(end 171.45 64.29375)
 		(stroke
